Commit message: adding docker compose

File: launch/include/config/robot.urdf.xacro (robot description, xacro)
@@ -13,5 +13,5 @@
     <parent link="chassis_link" />
     <child link="imu_link" />
-    <origin xyz="0 0 0" rpy="0 0 0" />
+    <origin xyz="0 0 0" rpy="0 0.00000003141592 0" />
   </joint>
   <link name="velodyne"> </link>
